Commit message: Extended arduinobot description for gazebo simulation

File: urdf/arduinobot.urdf.xacro (robot description, xacro)
@@ -5,4 +5,24 @@
     <xacro:property name="effort" value="30" />
     <xacro:property name="velocity" value="10" />
+    <xacro:macro name="default_inertial" params="mass">
+        <inertial>
+            <mass value="${mass}" />
+            <inertia ixx="1" ixy="0" ixz="0" iyy="1" iyz="0" izz="1" />
+        </inertial>
+    </xacro:macro>
+    <xacro:macro name="default_transmission" params="id">
+        <transmission name="transmission_${id}">
+            <type>
+                transmission_interface/SimpleTransmission
+            </type>
+            <joint name="joint_${id}">
+                <hardwareInterface>hardware_interface/PositionJointInterface</hardwareInterface>
+            </joint>
+            <actuator name="motor_${id}">
+                <hardwareInterface>hardware_interface/PositionJointInterface</hardwareInterface>
+                <mechanicalReduction>1</mechanicalReduction>
+            </actuator>
+        </transmission>
+    </xacro:macro>
     <!-- Links -->
     <link name="world" />
@@ -15,4 +35,12 @@
             </geometry>
         </visual>
+        <collision>
+            <origin rpy="0 0 0" xyz="-0.477 -0.5 0" />
+            <geometry>
+                <mesh filename="package://rr1_description/mesh/arduinobot/basement.stl"
+                    scale="0.01 0.01 0.01" />
+            </geometry>
+        </collision>
+        <xacro:default_inertial mass="1.0" />
     </link>
     <link name="base_plate">
@@ -24,4 +52,12 @@
             </geometry>
         </visual>
+        <collision>
+            <origin rpy="0 0 0" xyz="-0.357305 -0.4017354 -0.56" />
+            <geometry>
+                <mesh filename="package://rr1_description/mesh/arduinobot/base_plate.stl"
+                    scale="0.01 0.01 0.01" />
+            </geometry>
+        </collision>
+        <xacro:default_inertial mass="0.1" />
     </link>
     <link name="forward_drive_arm">
@@ -33,4 +69,12 @@
             </geometry>
         </visual>
+        <collision>
+            <origin rpy="0 -${PI/2} ${PI/2}" xyz="0.19 0.06 -0.08" />
+            <geometry>
+                <mesh filename="package://rr1_description/mesh/arduinobot/forward_drive_arm.stl"
+                    scale="0.01 0.01 0.01" />
+            </geometry>
+        </collision>
+        <xacro:default_inertial mass="0.1" />
     </link>
     <link name="horizontal_arm">
@@ -42,4 +86,12 @@
             </geometry>
         </visual>
+        <collision>
+            <origin rpy="${PI/2} 0 ${PI/2}" xyz="-0.03 -0.4 -0.06" />
+            <geometry>
+                <mesh filename="package://rr1_description/mesh/arduinobot/horizontal_arm.stl"
+                    scale="0.01 0.01 0.01" />
+            </geometry>
+        </collision>
+        <xacro:default_inertial mass="0.1" />
     </link>
     <link name="claw_support">
@@ -51,4 +103,12 @@
             </geometry>
         </visual>
+        <collision>
+            <origin rpy="0 0 ${PI/2}" xyz="0 -0.05 -0.15" />
+            <geometry>
+                <mesh filename="package://rr1_description/mesh/arduinobot/claw_support.stl"
+                    scale="0.01 0.01 0.01" />
+            </geometry>
+        </collision>
+        <xacro:default_inertial mass="0.05" />
     </link>
     <link name="gripper_right">
@@ -60,4 +120,12 @@
             </geometry>
         </visual>
+        <collision>
+            <origin rpy="0 0 -${PI/2}" xyz="-0.1 0.5 -0.1" />
+            <geometry>
+                <mesh filename="package://rr1_description/mesh/arduinobot/right_finger.stl"
+                    scale="0.01 0.01 0.01" />
+            </geometry>
+        </collision>
+        <xacro:default_inertial mass="0.01" />
     </link>
     <link name="gripper_left">
@@ -69,4 +137,12 @@
             </geometry>
         </visual>
+        <collision>
+            <origin rpy="0 0 -${PI/2}" xyz="-0.04 0.5 -0.1" />
+            <geometry>
+                <mesh filename="package://rr1_description/mesh/arduinobot/left_finger.stl"
+                    scale="0.01 0.01 0.01" />
+            </geometry>
+        </collision>
+        <xacro:default_inertial mass="0.01" />
     </link>
     <link name="tool_link" />
@@ -123,3 +199,23 @@
         <origin xyz="0 0 0" />
     </joint>
+    <xacro:default_transmission id="1" />
+    <xacro:default_transmission id="2" />
+    <xacro:default_transmission id="3" />
+    <xacro:default_transmission id="4" />
+    <gazebo>
+        <plugin name="gazebo_ros_control" filename="libgazebo_ros_control.so">
+            <robotNamespace>/arduinobot</robotNamespace>
+            <robotSimType>gazebo_ros_control/DefaultRobotHardwareSim</robotSimType>
+            <legacyModeNS>true</legacyModeNS>
+        </plugin>
+        <plugin name="joint_5_mimic_joint_4"
+            filename="libroboticsgroup_gazebo_mimic_joint_plugin.so">
+            <joint>joint_4</joint>
+            <mimicJoint>joint_5</mimicJoint>
+            <multiplier>-1.0</multiplier>
+            <offset>0</offset>
+            <maxEffort>${effort}</maxEffort>
+            <robotNamespace>/arduinobot</robotNamespace>
+        </plugin>
+    </gazebo>
 </robot>
