Commit message: Updated RR1 URDF to use the extended base meshes

File: urdf/rr1.urdf (robot description, URDF)
Before this commit: robot rr1, 8 links, 7 joints
Links:
- link base_link: mass 0.2 -> 0.5; geometry collision mesh filename=package://rr1_description/mesh/collision/01_RR1_extended_ba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 scale=0.001 0.001 0.001; visual mesh filename=package://rr1_description/mesh/visual/01_RR1_extended_base.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 scale=0.001 0.001 0.001

File: urdf/rr1.urdf.xacro (robot description, xacro)
@@ -15,7 +15,7 @@
     <link name="world" />
     <!-- Base -->
-    <xacro:rr1_link name="base_link" mesh_file="01_RR1_base">
+    <xacro:rr1_link name="base_link" mesh_file="01_RR1_extended_base">
         <origin rpy="0 0 0" xyz="-0.052 -0.013 0.179" />
-        <xacro:inertial_cylinder mass="0.2" r="0.073" h="0.075">
+        <xacro:inertial_cylinder mass="0.5" r="0.073" h="0.075">
             <origin rpy="0 0 0" xyz="0 0 0.0375" />
         </xacro:inertial_cylinder>
