Commit message: Finished URDF draft for RR1 visuals

File: urdf/rr1.urdf.xacro (robot description, xacro)
@@ -20,5 +20,5 @@
     <link name="shoulder_link">
         <visual>
-            <origin rpy="0 0 0" xyz="-0.052 -0.012986 0.109" />
+            <origin rpy="0 0 0" xyz="-0.052 -0.013 0.109" />
             <geometry>
                 <mesh filename="package://rr1_description/mesh/visual/02_RR1_shoulder.dae"
@@ -36,52 +36,40 @@
         </visual>
     </link>
-    <!-- <link name="elbow_link">
+    <link name="elbow_link">
         <visual>
-            <origin rpy="0 0 0"
-    xyz="${model_offset}" />
+            <origin rpy="0 0 0" xyz="0 -0.013 -0.225" />
             <geometry>
-                <mesh
-    filename="package://rr1_description/mesh/visual/04_RR1_elbow.dae"
-                    scale="${model_scale}"
-    />
+                <mesh filename="package://rr1_description/mesh/visual/04_RR1_elbow.dae"
+                    scale="${model_scale}" />
             </geometry>
         </visual>
-    </link> -->
-    <!-- <link name="forearm_link">
+    </link>
+    <link name="forearm_link">
         <visual>
-            <origin rpy="0 0 0"
-    xyz="${model_offset}" />
+            <origin rpy="0 0 0" xyz="0 -0.0042 -0.3257" />
             <geometry>
-                <mesh
-    filename="package://rr1_description/mesh/visual/05_RR1_forearm.dae"
-                    scale="${model_scale}"
-    />
+                <mesh filename="package://rr1_description/mesh/visual/05_RR1_forearm.dae"
+                    scale="${model_scale}" />
             </geometry>
         </visual>
-    </link> -->
-    <!-- <link name="wrist_link">
+    </link>
+    <link name="wrist_link">
         <visual>
-            <origin rpy="0 0 0"
-    xyz="${model_offset}" />
+            <origin rpy="0 0 0" xyz="0.284 -0.0042 -0.3257" />
             <geometry>
-                <mesh
-    filename="package://rr1_description/mesh/visual/06_RR1_wrist.dae"
-                    scale="${model_scale}"
-    />
+                <mesh filename="package://rr1_description/mesh/visual/06_RR1_wrist.dae"
+                    scale="${model_scale}" />
             </geometry>
         </visual>
-    </link> -->
-    <!-- <link name="hand_link">
+    </link>
+    <link name="hand_link">
         <visual>
-            <origin rpy="0 0 0"
-    xyz="${model_offset}" />
+            <origin rpy="0 0 0" xyz="0.284 -0.07 -0.3257" />
             <geometry>
-                <mesh
-    filename="package://rr1_description/mesh/visual/07_RR1_hand.dae"
-                    scale="${model_scale}"
-    />
+                <mesh filename="package://rr1_description/mesh/visual/07_RR1_hand.dae"
+                    scale="${model_scale}" />
             </geometry>
         </visual>
-    </link> -->
+    </link>
     <!-- Joints -->
     <joint name="virtual_joint" type="fixed">
@@ -104,27 +92,31 @@
         <limit lower="-${PI/2}" upper="${PI/2}" effort="${effort}" velocity="${velocity}" />
     </joint>
-    <!-- <joint name="joint_3" type="fixed">
+    <joint name="joint_3" type="revolute">
         <parent link="upper_arm_link" />
-        <child
-    link="elbow_link" />
-        <origin xyz="0 0 0" />
-    </joint> -->
-    <!-- <joint name="joint_4" type="fixed">
+        <child link="elbow_link" />
+        <origin xyz="0 0 0.225" />
+        <axis xyz="0 1 0" />
+        <limit lower="-${PI/2}" upper="${PI/2}" effort="${effort}" velocity="${velocity}" />
+    </joint>
+    <joint name="joint_4" type="revolute">
         <parent link="elbow_link" />
-        <child
-    link="forearm_link" />
-        <origin xyz="0 0 0" />
-    </joint> -->
-    <!-- <joint name="joint_5" type="fixed">
+        <child link="forearm_link" />
+        <origin xyz="0 -0.0088 0.1007" />
+        <axis xyz="1 0 0" />
+        <limit lower="-${PI/2}" upper="${PI/2}" effort="${effort}" velocity="${velocity}" />
+    </joint>
+    <joint name="joint_5" type="revolute">
         <parent link="forearm_link" />
-        <child
-    link="wrist_link" />
-        <origin xyz="0 0 0" />
-    </joint> -->
-    <!-- <joint name="joint_6" type="fixed">
+        <child link="wrist_link" />
+        <origin xyz="-0.284 0 0" />
+        <axis xyz="0 1 0" />
+        <limit lower="-${PI/8}" upper="${PI}" effort="${effort}" velocity="${velocity}" />
+    </joint>
+    <joint name="joint_6" type="revolute">
         <parent link="wrist_link" />
-        <child
-    link="hand_link" />
-        <origin xyz="0 0 0" />
-    </joint> -->
+        <child link="hand_link" />
+        <origin xyz="0 0.0658 0" />
+        <axis xyz="0 0 1" />
+        <limit lower="-${PI/2}" upper="${PI/2}" effort="${effort}" velocity="${velocity}" />
+    </joint>
 </robot>

Commit message: Removed meshes centered in the origin. Restructured URDF file for RR1 robot. Added some xacro includes.

File: urdf/rr1.urdf.xacro (robot description, xacro)
@@ -1,15 +1,17 @@
 <?xml version="1.0"?>
 <robot xmlns:xacro="http://www.ros.org/wiki/xacro" name="robot_name">
+    <!-- Includes -->
+    <xacro:include filename="includes/constants.xacro" />
+    <xacro:include filename="includes/inertial_macros.xacro" />
     <!-- Properties -->
-    <xacro:property name="PI" value="3.14159265359" />
     <xacro:property name="effort" value="30" />
     <xacro:property name="velocity" value="10" />
-    <xacro:property name="model_offset" value="-0.052 -0.012986 0.179" />
     <xacro:property name="model_scale" value="0.001 0.001 0.001" />
-    <!-- Links -->
+    <!-- We need a world link because we want the base link of the robot to be anchored to it -->
     <link name="world" />
+    <!-- Base -->
     <link name="base_link">
         <visual>
-            <origin rpy="0 0 0" xyz="${model_offset}" />
+            <origin rpy="0 0 0" xyz="-0.052 -0.013 0.179" />
             <geometry>
                 <mesh filename="package://rr1_description/mesh/visual/01_RR1_base.dae"
@@ -18,4 +20,10 @@
         </visual>
     </link>
+    <joint name="virtual_joint" type="fixed">
+        <parent link="world" />
+        <child link="base_link" />
+        <origin xyz="0 0 0" />
+    </joint>
+    <!-- Shoulder -->
     <link name="shoulder_link">
         <visual>
@@ -27,4 +35,12 @@
         </visual>
     </link>
+    <joint name="shoulder_joint" type="revolute">
+        <parent link="base_link" />
+        <child link="shoulder_link" />
+        <origin xyz="0 0 0.07" />
+        <axis xyz="0 0 1" />
+        <limit lower="-${PI}" upper="${PI}" effort="${effort}" velocity="${velocity}" />
+    </joint>
+    <!-- Upper Arm -->
     <link name="upper_arm_link">
         <visual>
@@ -36,4 +52,12 @@
         </visual>
     </link>
+    <joint name="upper_arm_joint" type="revolute">
+        <parent link="shoulder_link" />
+        <child link="upper_arm_link" />
+        <origin xyz="-0.052 0 0.109" />
+        <axis xyz="0 1 0" />
+        <limit lower="-${PI/2}" upper="${PI/2}" effort="${effort}" velocity="${velocity}" />
+    </joint>
+    <!-- Elbow -->
     <link name="elbow_link">
         <visual>
@@ -45,4 +69,12 @@
         </visual>
     </link>
+    <joint name="elbow_joint" type="revolute">
+        <parent link="upper_arm_link" />
+        <child link="elbow_link" />
+        <origin xyz="0 0 0.225" />
+        <axis xyz="0 1 0" />
+        <limit lower="-${PI/2}" upper="${PI/2}" effort="${effort}" velocity="${velocity}" />
+    </joint>
+    <!-- Forearm -->
     <link name="forearm_link">
         <visual>
@@ -54,4 +86,12 @@
         </visual>
     </link>
+    <joint name="forearm_link" type="revolute">
+        <parent link="elbow_link" />
+        <child link="forearm_link" />
+        <origin xyz="0 -0.0088 0.1007" />
+        <axis xyz="1 0 0" />
+        <limit lower="-${PI/2}" upper="${PI/2}" effort="${effort}" velocity="${velocity}" />
+    </joint>
+    <!-- Wrist -->
     <link name="wrist_link">
         <visual>
@@ -63,4 +103,12 @@
         </visual>
     </link>
+    <joint name="wrist_joint" type="revolute">
+        <parent link="forearm_link" />
+        <child link="wrist_link" />
+        <origin xyz="-0.284 0 0" />
+        <axis xyz="0 1 0" />
+        <limit lower="-${PI/8}" upper="${PI}" effort="${effort}" velocity="${velocity}" />
+    </joint>
+    <!-- Hand -->
     <link name="hand_link">
         <visual>
@@ -72,46 +120,5 @@
         </visual>
     </link>
-    <!-- Joints -->
-    <joint name="virtual_joint" type="fixed">
-        <parent link="world" />
-        <child link="base_link" />
-        <origin xyz="0 0 0" />
-    </joint>
-    <joint name="joint_1" type="revolute">
-        <parent link="base_link" />
-        <child link="shoulder_link" />
-        <origin xyz="0 0 0.07" />
-        <axis xyz="0 0 1" />
-        <limit lower="-${PI}" upper="${PI}" effort="${effort}" velocity="${velocity}" />
-    </joint>
-    <joint name="joint_2" type="revolute">
-        <parent link="shoulder_link" />
-        <child link="upper_arm_link" />
-        <origin xyz="-0.052 0 0.109" />
-        <axis xyz="0 1 0" />
-        <limit lower="-${PI/2}" upper="${PI/2}" effort="${effort}" velocity="${velocity}" />
-    </joint>
-    <joint name="joint_3" type="revolute">
-        <parent link="upper_arm_link" />
-        <child link="elbow_link" />
-        <origin xyz="0 0 0.225" />
-        <axis xyz="0 1 0" />
-        <limit lower="-${PI/2}" upper="${PI/2}" effort="${effort}" velocity="${velocity}" />
-    </joint>
-    <joint name="joint_4" type="revolute">
-        <parent link="elbow_link" />
-        <child link="forearm_link" />
-        <origin xyz="0 -0.0088 0.1007" />
-        <axis xyz="1 0 0" />
-        <limit lower="-${PI/2}" upper="${PI/2}" effort="${effort}" velocity="${velocity}" />
-    </joint>
-    <joint name="joint_5" type="revolute">
-        <parent link="forearm_link" />
-        <child link="wrist_link" />
-        <origin xyz="-0.284 0 0" />
-        <axis xyz="0 1 0" />
-        <limit lower="-${PI/8}" upper="${PI}" effort="${effort}" velocity="${velocity}" />
-    </joint>
-    <joint name="joint_6" type="revolute">
+    <joint name="hand_joint" type="revolute">
         <parent link="wrist_link" />
         <child link="hand_link" />

Commit message: Added ros2_control and gazebo tags to the description, added dynamics to the joints, small fixes in link/joint names

File: urdf/rr1.urdf.xacro (robot description, xacro)
@@ -5,7 +5,10 @@
     <xacro:include filename="includes/inertial_macros.xacro" />
     <xacro:include filename="includes/custom_macros.xacro" />
+    <xacro:include filename="includes/ros2_control.xacro" />
     <!-- Properties -->
     <xacro:property name="effort" value="30" />
     <xacro:property name="velocity" value="10" />
+    <xacro:property name="damping" value="10" />
+    <xacro:property name="friction" value="10.0" />
     <xacro:property name="model_scale" value="0.001 0.001 0.001" />
     <!-- We need a world link because we want the base link of the robot to be anchored to it -->
@@ -36,4 +39,5 @@
         <axis xyz="0 0 1" />
         <limit lower="-${PI}" upper="${PI}" effort="${effort}" velocity="${velocity}" />
+        <dynamics damping="${damping}" friction="${friction}" />
     </joint>
     <!-- Upper Arm -->
@@ -50,4 +54,5 @@
         <axis xyz="0 1 0" />
         <limit lower="-${PI/2}" upper="${PI/2}" effort="${effort}" velocity="${velocity}" />
+        <dynamics damping="${damping}" friction="${friction}" />
     </joint>
     <!-- Elbow -->
@@ -64,4 +69,5 @@
         <axis xyz="0 1 0" />
         <limit lower="-${PI/2}" upper="${PI/2}" effort="${effort}" velocity="${velocity}" />
+        <dynamics damping="${damping}" friction="${friction}" />
     </joint>
     <!-- Forearm -->
@@ -72,5 +78,5 @@
         </xacro:inertial_cylinder>
     </xacro:rr1_link>
-    <joint name="forearm_link" type="revolute">
+    <joint name="forearm_joint" type="revolute">
         <parent link="elbow_link" />
         <child link="forearm_link" />
@@ -78,4 +84,5 @@
         <axis xyz="1 0 0" />
         <limit lower="-${PI/2}" upper="${PI/2}" effort="${effort}" velocity="${velocity}" />
+        <dynamics damping="${damping}" friction="${friction}" />
     </joint>
     <!-- Wrist -->
@@ -92,4 +99,5 @@
         <axis xyz="0 1 0" />
         <limit lower="-${PI/8}" upper="${PI}" effort="${effort}" velocity="${velocity}" />
+        <dynamics damping="${damping}" friction="${friction}" />
     </joint>
     <!-- Hand -->
@@ -106,4 +114,5 @@
         <axis xyz="0 0 1" />
         <limit lower="-${PI/2}" upper="${PI/2}" effort="${effort}" velocity="${velocity}" />
+        <dynamics damping="${damping}" friction="${friction}" />
     </joint>
 </robot>

Commit message: Updated inertial of the base link

File: urdf/rr1.urdf.xacro (robot description, xacro)
@@ -19,7 +19,7 @@
     <xacro:rr1_link name="base_link" mesh_file="01_RR1_extended_base">
         <origin rpy="0 0 0" xyz="-0.052 -0.013 0.179" />
-        <xacro:inertial_cylinder mass="0.5" r="0.073" h="0.075">
-            <origin rpy="0 0 0" xyz="0 0 0.0375" />
-        </xacro:inertial_cylinder>
+        <xacro:inertial_box mass="0.5" x="0.36" y="0.15" z="0.09">
+            <origin rpy="0 0 0" xyz="0.105 0 0.0375" />
+        </xacro:inertial_box>
     </xacro:rr1_link>
     <joint name="virtual_joint" type="fixed">
