Commit message: Finalized urdf with gripper

File: urdf/includes/ros2_control.xacro (robot description, xacro)
@@ -66,4 +66,13 @@
             <state_interface name="effort" />
         </joint>
+        <joint name="finger_joint">
+            <command_interface name="position">
+                <param name="min">-0.04</param>
+                <param name="max">0.785</param>
+            </command_interface>
+            <state_interface name="position" />
+            <state_interface name="velocity" />
+            <state_interface name="effort" />
+        </joint>
     </ros2_control>
 </robot>

File: urdf/rr1.urdf (robot description, URDF)
Before this commit: robot rr1, 8 links, 7 joints
Links:
- added link finger_link, mass 0.02; collision mesh filename=package://rr1_description/mesh/collision/08_RR1_grip.stl scale=0.001 0.001 0.001; visual mesh filename=package://rr1_description/mesh/visual/08_RR1_grip.dae scale=0.001 0.001 0.001
- added link opposite_finger_link, mass 0.02; collision mesh filename=package://rr1_description/mesh/collision/08_RR1_grip_opposi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 scale=0.001 0.001 0.001; visual mesh filename=package://rr1_description/mesh/visual/08_RR1_grip_opposite.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 scale=0.001 0.001 0.001
- added link tool
- link hand_link: geometry collision mesh filename=package://rr1_description/mesh/collision/07_RR1_hand_no_gri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 scale=0.001 0.001 0.001; visual mesh filename=package://rr1_description/mesh/visual/07_RR1_hand_no_grip.d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 scale=0.001 0.001 0.001
Joints:
- added joint finger_joint: type revolute, parent hand_link, child finger_link, origin xyz=0.01 0 -0.15, axis 0 -1 0, limit lower=-0.04 upper=0.7853981633975 effort=30 velocity=10
- added joint opposite_finger_joint: type revolute, parent hand_link, child opposite_finger_link, origin xyz=-0.01 0 -0.15, axis 0 1 0, limit lower=-0.04 upper=0.7853981633975 effort=30 velocity=10, mimic joint=finger_joint
- added joint tool_joint: type fixed, parent hand_link, child tool, origin xyz=0 0 -0.195

File: urdf/rr1.urdf.xacro (robot description, xacro)
@@ -102,8 +102,8 @@
     </joint>
     <!-- Hand -->
-    <xacro:rr1_link name="hand_link" mesh_file="07_RR1_hand">
+    <xacro:rr1_link name="hand_link" mesh_file="07_RR1_hand_no_grip">
         <origin rpy="0 0 0" xyz="0.284 -0.07 -0.3257" />
-        <xacro:inertial_cylinder mass="0.2" r="0.0375" h="0.2">
-            <origin rpy="0 0 0" xyz="0 0 -0.11" />
+        <xacro:inertial_cylinder mass="0.2" r="0.0375" h="0.14">
+            <origin rpy="0 0 0" xyz="0 0 -0.08" />
         </xacro:inertial_cylinder>
     </xacro:rr1_link>
@@ -116,3 +116,39 @@
         <dynamics damping="${damping}" friction="${friction}" />
     </joint>
+    <!-- Gripper -->
+    <xacro:rr1_link name="finger_link" mesh_file="08_RR1_grip">
+        <origin rpy="0 0 0" xyz="0.274 -0.07 -0.1757" />
+        <xacro:inertial_box mass="0.02" x="0.01" y="0.02" z="0.06">
+            <origin rpy="0 0 0" xyz="0.01 0 -0.05" />
+        </xacro:inertial_box>
+    </xacro:rr1_link>
+    <joint name="finger_joint" type="revolute">
+        <parent link="hand_link" />
+        <child link="finger_link" />
+        <origin xyz="0.01 0 -0.15" />
+        <axis xyz="0 -1 0" />
+        <limit lower="-0.04" upper="${PI/4}" effort="${effort}" velocity="${velocity}" />
+        <dynamics damping="${damping}" friction="${friction}" />
+    </joint>
+    <xacro:rr1_link name="opposite_finger_link" mesh_file="08_RR1_grip_opposite">
+        <origin rpy="0 0 0" xyz="0.294 -0.07 -0.1757" />
+        <xacro:inertial_box mass="0.02" x="0.01" y="0.02" z="0.06">
+            <origin rpy="0 0 0" xyz="-0.01 0 -0.05" />
+        </xacro:inertial_box>
+    </xacro:rr1_link>
+    <joint name="opposite_finger_joint" type="revolute">
+        <parent link="hand_link" />
+        <child link="opposite_finger_link" />
+        <origin xyz="-0.01 0 -0.15" />
+        <axis xyz="0 1 0" />
+        <mimic joint="finger_joint" />
+        <limit lower="-0.04" upper="${PI/4}" effort="${effort}" velocity="${velocity}" />
+        <dynamics damping="${damping}" friction="${friction}" />
+    </joint>
+    <link name="tool" />
+    <joint name="tool_joint" type="fixed">
+        <parent link="hand_link" />
+        <child link="tool" />
+        <origin xyz="0 0 -0.195" />
+    </joint>
 </robot>

Commit message: Fixed controller configuration for grippers

File: urdf/includes/ros2_control.xacro (robot description, xacro)
@@ -75,4 +75,12 @@
             <state_interface name="effort" />
         </joint>
+        <joint name="opposite_finger_joint">
+            <param name="mimic">finger_joint</param>
+            <param name="multiplier">-1</param>
+            <command_interface name="position" />
+            <state_interface name="position" />
+            <state_interface name="velocity" />
+            <state_interface name="effort" />
+        </joint>
     </ros2_control>
 </robot>
