Commit message: Updated mass and limit estimations for RR1, created macro for ros2_control_joint blocks

File: urdf/includes/constants.xacro (robot description, xacro)
@@ -3,3 +3,4 @@
     <!-- Common mathematical constants -->
     <xacro:property name="PI" value="3.14159265359" />
+    <xacro:property name="RPM_TO_RAD_S" value="0.1047198" />
 </robot>

File: urdf/includes/custom_macros.xacro (robot description, xacro)
@@ -24,3 +24,20 @@
         </link>
     </xacro:macro>
+    <xacro:macro name="ros2_control_joint" params="name min_lim max_lim">
+        <joint name="${name}">
+            <command_interface name="position">
+                <param name="min">${min_lim}</param>
+                <param name="max">${max_lim}</param>
+            </command_interface>
+            <state_interface name="position">
+                <param name="initial_value">0.0</param>
+            </state_interface>
+            <state_interface name="velocity">
+                <param name="initial_value">0.0</param>
+            </state_interface>
+            <state_interface name="effort">
+                <param name="initial_value">0.0</param>
+            </state_interface>
+        </joint>
+    </xacro:macro>
 </robot>

File: urdf/includes/ros2_control.xacro (robot description, xacro)
@@ -16,124 +16,20 @@
             <plugin>gazebo_ros2_control/GazeboSystem</plugin>
         </hardware>
-        <joint name="shoulder_joint">
-            <command_interface name="position">
-                <param name="min">-3.14</param>
-                <param name="max">3.14</param>
-            </command_interface>
-            <state_interface name="position">
-                <param name="initial_value">0.0</param>
-            </state_interface>
-            <state_interface name="velocity">
-                <param name="initial_value">0.0</param>
-            </state_interface>
-            <state_interface name="effort">
-                <param name="initial_value">0.0</param>
-            </state_interface>
-        </joint>
-        <joint name="upper_arm_joint">
-            <command_interface name="position">
-                <param name="min">-3.14</param>
-                <param name="max">3.14</param>
-            </command_interface>
-            <state_interface name="position">
-                <param name="initial_value">0.0</param>
-            </state_interface>
-            <state_interface name="velocity">
-                <param name="initial_value">0.0</param>
-            </state_interface>
-            <state_interface name="effort">
-                <param name="initial_value">0.0</param>
-            </state_interface>
-        </joint>
-        <joint name="elbow_joint">
-            <command_interface name="position">
-                <param name="min">-3.14</param>
-                <param name="max">3.14</param>
-            </command_interface>
-            <state_interface name="position">
-                <param name="initial_value">0.0</param>
-            </state_interface>
-            <state_interface name="velocity">
-                <param name="initial_value">0.0</param>
-            </state_interface>
-            <state_interface name="effort">
-                <param name="initial_value">0.0</param>
-            </state_interface>
-        </joint>
-        <joint name="forearm_joint">
-            <command_interface name="position">
-                <param name="min">-3.14</param>
-                <param name="max">3.14</param>
-            </command_interface>
-            <state_interface name="position">
-                <param name="initial_value">0.0</param>
-            </state_interface>
-            <state_interface name="velocity">
-                <param name="initial_value">0.0</param>
-            </state_interface>
-            <state_interface name="effort">
-                <param name="initial_value">0.0</param>
-            </state_interface>
-        </joint>
-        <joint name="wrist_joint">
-            <command_interface name="position">
-                <param name="min">-3.14</param>
-                <param name="max">3.14</param>
-            </command_interface>
-            <state_interface name="position">
-                <param name="initial_value">0.0</param>
-            </state_interface>
-            <state_interface name="velocity">
-                <param name="initial_value">0.0</param>
-            </state_interface>
-            <state_interface name="effort">
-                <param name="initial_value">0.0</param>
-            </state_interface>
-        </joint>
-        <joint name="hand_joint">
-            <command_interface name="position">
-                <param name="min">-3.14</param>
-                <param name="max">3.14</param>
-            </command_interface>
-            <state_interface name="position">
-                <param name="initial_value">0.0</param>
-            </state_interface>
-            <state_interface name="velocity">
-                <param name="initial_value">0.0</param>
-            </state_interface>
-            <state_interface name="effort">
-                <param name="initial_value">0.0</param>
-            </state_interface>
-        </joint>
-        <joint name="finger_joint">
-            <command_interface name="position">
-                <param name="min">-0.04</param>
-                <param name="max">0.785</param>
-            </command_interface>
-            <state_interface name="position">
-                <param name="initial_value">0.0</param>
-            </state_interface>
-            <state_interface name="velocity">
-                <param name="initial_value">0.0</param>
-            </state_interface>
-            <state_interface name="effort">
-                <param name="initial_value">0.0</param>
-            </state_interface>
-        </joint>
-        <joint name="opposite_finger_joint">
-            <command_interface name="position">
-                <param name="min">-0.04</param>
-                <param name="max">0.785</param>
-            </command_interface>
-            <state_interface name="position">
-                <param name="initial_value">0.0</param>
-            </state_interface>
-            <state_interface name="velocity">
-                <param name="initial_value">0.0</param>
-            </state_interface>
-            <state_interface name="effort">
-                <param name="initial_value">0.0</param>
-            </state_interface>
-        </joint>
+        <xacro:ros2_control_joint name="shoulder_joint"
+            min_lim="-${PI*3/4}" max_lim="${PI*3/4}" />
+        <xacro:ros2_control_joint name="upper_arm_joint"
+            min_lim="-${PI/8}" max_lim="${PI/8}" />
+        <xacro:ros2_control_joint name="elbow_joint"
+            min_lim="-${PI/2}" max_lim="${PI/2}" />
+        <xacro:ros2_control_joint name="forearm_joint"
+            min_lim="-${PI*3/4}" max_lim="${PI*3/4}" />
+        <xacro:ros2_control_joint name="wrist_joint"
+            min_lim="0" max_lim="${PI}" />
+        <xacro:ros2_control_joint name="hand_joint"
+            min_lim="-${PI*3/4}" max_lim="${PI*3/4}" />
+        <xacro:ros2_control_joint name="finger_joint"
+            min_lim="0" max_lim="${PI*3/8}" />
+        <xacro:ros2_control_joint name="opposite_finger_joint"
+            min_lim="0" max_lim="${PI*3/8}" />
     </ros2_control>
 </robot>

File: urdf/rr1.urdf (robot description, URDF)
Before this commit: robot rr1, 11 links, 10 joints
Links:
- link base_link: mass 0.5 -> 4.0
- link elbow_link: mass 0.3 -> 1.75
- link finger_link: mass 0.02 -> 0.25
- link forearm_link: mass 0.35 -> 1.5
- link hand_link: mass 0.2 -> 0.5
- link opposite_finger_link: mass 0.02 -> 0.25
- link shoulder_link: mass 0.2 -> 2.5
- link upper_arm_link: mass 0.4 -> 2.5
- link wrist_link: mass 0.15 -> 1.0
Joints:
- joint elbow_joint: limit lower=-1.570796326795 upper=1.570796326795 effort=30 velocity=10 -> lower=-1.570796326795 upper=1.570796326795 effort=30 velocity=7.853985
- joint finger_joint: limit lower=-0.04 upper=0.7853981633975 effort=30 velocity=10 -> lower=0 upper=1.1780972450962501 effort=30 velocity=7.853985
- joint forearm_joint: limit lower=-1.570796326795 upper=1.570796326795 effort=30 velocity=10 -> lower=-2.3561944901925003 upper=2.3561944901925003 effort=30 velocity=7.853985
- joint hand_joint: limit lower=-1.570796326795 upper=1.570796326795 effort=30 velocity=10 -> lower=-2.3561944901925003 upper=2.3561944901925003 effort=30 velocity=7.853985
- joint opposite_finger_joint: limit lower=-0.04 upper=0.7853981633975 effort=30 velocity=10 -> lower=0 upper=1.1780972450962501 effort=30 velocity=7.853985
- joint shoulder_joint: limit lower=-3.14159265359 upper=3.14159265359 effort=30 velocity=10 -> lower=-2.3561944901925003 upper=2.3561944901925003 effort=30 velocity=7.853985
- joint upper_arm_joint: limit lower=-1.570796326795 upper=1.570796326795 effort=30 velocity=10 -> lower=-0.39269908169875 upper=0.39269908169875 effort=30 velocity=7.853985
- joint wrist_joint: limit lower=-0.39269908169875 upper=3.14159265359 effort=30 velocity=10 -> lower=0 upper=3.14159265359 effort=30 velocity=7.853985

File: urdf/rr1.urdf.xacro (robot description, xacro)
@@ -10,7 +10,8 @@
     <!-- Properties -->
     <xacro:property name="effort" value="30" />
-    <xacro:property name="velocity" value="10" />
+    <xacro:property name="rpm" value="75" /> <!-- Including transmission-->
     <xacro:property name="damping" value="10" />
     <xacro:property name="friction" value="10.0" />
+    <xacro:property name="velocity" value="${rpm * RPM_TO_RAD_S}" />
     <xacro:property name="model_scale" value="0.001 0.001 0.001" />
     <!-- We need a world link because we want the base link of the robot to be anchored to it -->
@@ -19,5 +20,5 @@
     <xacro:rr1_link name="base_link" mesh_file="01_RR1_extended_base">
         <origin rpy="0 0 0" xyz="-0.052 -0.013 0.179" />
-        <xacro:inertial_box mass="0.5" x="0.36" y="0.15" z="0.09">
+        <xacro:inertial_box mass="4.0" x="0.36" y="0.15" z="0.09">
             <origin rpy="0 0 0" xyz="0.105 0 0.0375" />
         </xacro:inertial_box>
@@ -31,5 +32,5 @@
     <xacro:rr1_link name="shoulder_link" mesh_file="02_RR1_shoulder">
         <origin rpy="0 0 0" xyz="-0.052 -0.013 0.109" />
-        <xacro:inertial_cylinder mass="0.2" r="0.05" h="0.18">
+        <xacro:inertial_cylinder mass="2.5" r="0.05" h="0.18">
             <origin rpy="0 -${PI/8} 0" xyz="-0.04 -0.035 0.0545" />
         </xacro:inertial_cylinder>
@@ -40,5 +41,5 @@
         <origin xyz="0 0 0.07" />
         <axis xyz="0 0 1" />
-        <limit lower="-${PI}" upper="${PI}" effort="${effort}" velocity="${velocity}" />
+        <limit lower="-${PI*3/4}" upper="${PI*3/4}" effort="${effort}" velocity="${velocity}" />
         <dynamics damping="${damping}" friction="${friction}" />
     </joint>
@@ -46,5 +47,5 @@
     <xacro:rr1_link name="upper_arm_link" mesh_file="03_RR1_upper_arm">
         <origin rpy="0 0 0" xyz="0 -0.013 0" />
-        <xacro:inertial_cylinder mass="0.4" r="0.085" h="0.32">
+        <xacro:inertial_cylinder mass="2.5" r="0.085" h="0.32">
             <origin rpy="0 0 0" xyz="0 0.035 0.125" />
         </xacro:inertial_cylinder>
@@ -55,5 +56,5 @@
         <origin xyz="-0.052 0 0.109" />
         <axis xyz="0 1 0" />
-        <limit lower="-${PI/2}" upper="${PI/2}" effort="${effort}" velocity="${velocity}" />
+        <limit lower="-${PI/8}" upper="${PI/8}" effort="${effort}" velocity="${velocity}" />
         <dynamics damping="${damping}" friction="${friction}" />
     </joint>
@@ -61,5 +62,5 @@
     <xacro:rr1_link name="elbow_link" mesh_file="04_RR1_elbow">
         <origin rpy="0 0 0" xyz="0 -0.013 -0.225" />
-        <xacro:inertial_box mass="0.3" x="0.174" y="0.055" z="0.19">
+        <xacro:inertial_box mass="1.75" x="0.174" y="0.055" z="0.19">
             <origin rpy="0 0 0" xyz="0.032 0 0.04" />
         </xacro:inertial_box>
@@ -76,5 +77,5 @@
     <xacro:rr1_link name="forearm_link" mesh_file="05_RR1_forearm">
         <origin rpy="0 0 0" xyz="0 -0.0042 -0.3257" />
-        <xacro:inertial_cylinder mass="0.35" r="0.05" h="0.26">
+        <xacro:inertial_cylinder mass="1.5" r="0.05" h="0.26">
             <origin rpy="0 -${PI/2} 0" xyz="-0.18 0 0" />
         </xacro:inertial_cylinder>
@@ -85,5 +86,5 @@
         <origin xyz="0 -0.0088 0.1007" />
         <axis xyz="1 0 0" />
-        <limit lower="-${PI/2}" upper="${PI/2}" effort="${effort}" velocity="${velocity}" />
+        <limit lower="-${PI*3/4}" upper="${PI*3/4}" effort="${effort}" velocity="${velocity}" />
         <dynamics damping="${damping}" friction="${friction}" />
     </joint>
@@ -91,5 +92,5 @@
     <xacro:rr1_link name="wrist_link" mesh_file="06_RR1_wrist">
         <origin rpy="0 0 0" xyz="0.284 -0.0042 -0.3257" />
-        <xacro:inertial_box mass="0.15" x="0.044" y="0.044" z="0.11">
+        <xacro:inertial_box mass="1.0" x="0.044" y="0.044" z="0.11">
             <origin rpy="0 0 0" xyz="0 0.062 0.038" />
         </xacro:inertial_box>
@@ -100,5 +101,5 @@
         <origin xyz="-0.284 0 0" />
         <axis xyz="0 1 0" />
-        <limit lower="-${PI/8}" upper="${PI}" effort="${effort}" velocity="${velocity}" />
+        <limit lower="0" upper="${PI}" effort="${effort}" velocity="${velocity}" />
         <dynamics damping="${damping}" friction="${friction}" />
     </joint>
@@ -106,5 +107,5 @@
     <xacro:rr1_link name="hand_link" mesh_file="07_RR1_hand_no_grip">
         <origin rpy="0 0 0" xyz="0.284 -0.07 -0.3257" />
-        <xacro:inertial_cylinder mass="0.2" r="0.0375" h="0.14">
+        <xacro:inertial_cylinder mass="0.5" r="0.0375" h="0.14">
             <origin rpy="0 0 0" xyz="0 0 -0.08" />
         </xacro:inertial_cylinder>
@@ -115,5 +116,5 @@
         <origin xyz="0 0.0658 0" />
         <axis xyz="0 0 1" />
-        <limit lower="-${PI/2}" upper="${PI/2}" effort="${effort}" velocity="${velocity}" />
+        <limit lower="-${PI*3/4}" upper="${PI*3/4}" effort="${effort}" velocity="${velocity}" />
         <dynamics damping="${damping}" friction="${friction}" />
     </joint>
@@ -121,5 +122,5 @@
     <xacro:rr1_link name="finger_link" mesh_file="08_RR1_grip">
         <origin rpy="0 0 0" xyz="0.274 -0.07 -0.1757" />
-        <xacro:inertial_box mass="0.02" x="0.01" y="0.02" z="0.06">
+        <xacro:inertial_box mass="0.25" x="0.01" y="0.02" z="0.06">
             <origin rpy="0 0 0" xyz="0.01 0 -0.05" />
         </xacro:inertial_box>
@@ -130,10 +131,10 @@
         <origin xyz="0.01 0 -0.15" />
         <axis xyz="0 -1 0" />
-        <limit lower="-0.04" upper="${PI/4}" effort="${effort}" velocity="${velocity}" />
+        <limit lower="0" upper="${PI*3/8}" effort="${effort}" velocity="${velocity}" />
         <dynamics damping="${damping}" friction="${friction}" />
     </joint>
     <xacro:rr1_link name="opposite_finger_link" mesh_file="08_RR1_grip_opposite">
         <origin rpy="0 0 0" xyz="0.294 -0.07 -0.1757" />
-        <xacro:inertial_box mass="0.02" x="0.01" y="0.02" z="0.06">
+        <xacro:inertial_box mass="0.25" x="0.01" y="0.02" z="0.06">
             <origin rpy="0 0 0" xyz="-0.01 0 -0.05" />
         </xacro:inertial_box>
@@ -145,5 +146,5 @@
         <axis xyz="0 1 0" />
         <mimic joint="finger_joint" />
-        <limit lower="-0.04" upper="${PI/4}" effort="${effort}" velocity="${velocity}" />
+        <limit lower="0" upper="${PI*3/8 }" effort="${effort}" velocity="${velocity}" />
         <dynamics damping="${damping}" friction="${friction}" />
     </joint>
